Commit message: Changed size of chasis

File: description/robot_core.xacro (robot description, xacro)
@@ -22,7 +22,7 @@
     <link name="chasis">
         <visual>
-        <origin xyz="0.0075 0 0.0315"/>
+        <origin xyz="0.075 0 0.315"/>
             <geometry>
-                <box size="0.015 0.023 0.063"/>
+                <box size="0.15 0.23 0.63"/>
             </geometry>
             <material name="white"/>

Commit message: Updated Xacro's

File: description/robot_core.xacro (robot description, xacro)
@@ -1,4 +1,5 @@
 <?xml version="1.0"?>
 <robot xmlns:xacro="http://www.ros.org/wiki/xacro"  name="robot">
+    <xacro:include filename="inertial_macros.xacro"/>
    <material name="white">
         <color rgba="1 1 1 1"/>
@@ -13,19 +14,102 @@
         <color rgba="0 0 0 1"/>
    </material>
+    <!---Base-LInk-->
    <link name="base_link">
    </link>
+   <!---Chasis-LInk-->
     <joint name="chasis_joint" type="fixed">
     <parent link="base_link"/>
     <child link="chasis"/>
-    <origin xyz="-0.1 0 0"/>
+    <origin xyz="-0.13 0 0"/>
     </joint>
     <link name="chasis">
         <visual>
-        <origin xyz="0.075 0 0.315"/>
+        <origin xyz="0.075 0 0.0315"/>
             <geometry>
-                <box size="0.15 0.23 0.63"/>
+                <box size="0.15 0.23 0.063"/>
             </geometry>
             <material name="white"/>
         </visual>
+        <collision>
+        <origin xyz="0.075 0 0.0315"/>
+            <geometry>
+                <box size="0.15 0.23 0.063"/>
+            </geometry>
+            <material name="white"/>
+        </collision>
+        <xacro:inertial_box mass="0.5" x="0.15" y="0.23" z="0.063">
+            <origin xyz="0.075 0 0.0315" rpy="0 0 0"/>
+        </xacro:inertial_box>
+    </link>
+    <!--Left-Wheel-Link-->
+    <joint name="left_wheel_joint" type="continuous">
+        <parent link ="base_link"/>
+        <child link = "left_wheel"/>
+        <origin xyz="0 0.165 0" rpy="-${pi/2} 0 0"/>
+        <axis xyz="0 0 1"/>
+    </joint>
+    <link name = "left_wheel">
+    <visual>
+        <geometry>
+            <cylinder radius="0.04" length="0.04"/>
+        </geometry>
+        <material name="blue"/>
+    </visual>
+    <collision>
+        <geometry>
+            <cylinder radius="0.04" length="0.04"/>
+        </geometry>
+        <material name="blue"/>
+    </collision>
+    <xacro:inertial_cylinder mass="0.1" length="0.04" radius="0.04">
+        <origin xyz="0 0 0" rpy="0 0 0"/>
+    </xacro:inertial_cylinder>
+    </link>
+    <!--Right-Wheel-Link-->
+    <joint name="right_wheel_joint" type="continuous">
+        <parent link ="base_link"/>
+        <child link = "right_wheel"/>
+        <origin xyz="0 -0.165 0" rpy="${pi/2} 0 0"/>
+        <axis xyz="0 0 1"/>
+    </joint>
+    <link name = "right_wheel">
+    <visual>
+        <geometry>
+            <cylinder radius="0.04" length="0.04"/>
+        </geometry>
+        <material name="blue"/>
+    </visual>
+    <collision>
+        <geometry>
+            <cylinder radius="0.04" length="0.04"/>
+        </geometry>
+        <material name="blue"/>
+    </collision>
+    <xacro:inertial_cylinder mass="0.1" length="0.04" radius="0.04">
+        <origin xyz="0 0 0" rpy="0 0 0"/>
+    </xacro:inertial_cylinder>
+    </link>
+    <!--Caster Wheel-->
+    <joint name="caster_wheel_joint" type="fixed">
+        <parent link="base_link"/>
+        <child link="caster_wheel"/>
+        <origin xyz="-0.13 0 0"/>
+    </joint>
+    <link name="caster_wheel">
+    <visual>
+        <geometry>
+            <sphere radius="0.02"/>
+        </geometry>
+        <material name="black"/>
+    </visual>
+     <collision>
+        <geometry>
+            <sphere radius="0.02"/>
+        </geometry>
+        <material name="black"/>
+    </collision>
+    <xacro:inertial_sphere mass="0.1" radius="0.05">
+        <origin xyz="0 0 0" rpy="0 0 0"/>
+    </xacro:inertial_sphere>
     </link>
 </robot>

Commit message: Added Gazebo basic Simulation

File: description/robot_core.xacro (robot description, xacro)
@@ -42,9 +42,12 @@
         </xacro:inertial_box>
     </link>
+    <gazebo reference="chasis">
+        <material>Gazebo/White</material>
+    </gazebo>
     <!--Left-Wheel-Link-->
     <joint name="left_wheel_joint" type="continuous">
         <parent link ="base_link"/>
         <child link = "left_wheel"/>
-        <origin xyz="0 0.165 0" rpy="-${pi/2} 0 0"/>
+        <origin xyz="0 0.165 0" rpy="${pi/2} 0 0"/>
         <axis xyz="0 0 1"/>
     </joint>
@@ -66,4 +69,7 @@
     </xacro:inertial_cylinder>
     </link>
+    <gazebo reference="left_wheel">
+        <material>Gazebo/Blue</material>
+    </gazebo>
     <!--Right-Wheel-Link-->
     <joint name="right_wheel_joint" type="continuous">
@@ -90,9 +96,12 @@
     </xacro:inertial_cylinder>
     </link>
+    <gazebo reference="right_wheel">
+        <material>Gazebo/Blue</material>
+    </gazebo>
     <!--Caster Wheel-->
     <joint name="caster_wheel_joint" type="fixed">
         <parent link="base_link"/>
         <child link="caster_wheel"/>
-        <origin xyz="-0.13 0 0"/>
+        <origin xyz="-0.13 0 -0.018"/>
     </joint>
     <link name="caster_wheel">
@@ -113,3 +122,8 @@
     </xacro:inertial_sphere>
     </link>
+    <gazebo reference="caster_wheel">
+        <material>Gazebo/Black</material>
+        <mu1 value="0.001"/>
+        <mu2 value="0.001"/>
+    </gazebo>
 </robot>

Commit message: Localization Added

File: description/robot_core.xacro (robot description, xacro)
@@ -19,4 +19,12 @@
     <!---Base-LInk-->
    <link name="base_link">
+   </link>
+   <!--Base FootPrint Link-->
+   <joint name="base_footprint_joint" type="fixed">
+    <parent link="base_link"/>
+    <child link="base_footprint"/>
+    <origin xyz="0 0 0" rpy="0 0 0"/>
+   </joint>
+   <link name="base_footprint">
    </link>
    <!---Chasis-LInk-->
@@ -130,3 +138,28 @@
         <mu2 value="0.001"/>
     </gazebo>
+    <!-- IMU Sensor -->
+    <joint name="base_to_imu" type="fixed">
+        <parent link="base_link"/>
+        <child link="imu"/>
+        <origin xyz="0 0 0.1" rpy="0 0 0"/>
+    </joint>
+    <link name="imu">
+        <visual>
+            <geometry>
+                <box size="0.03 0.03 0.03"/>
+            </geometry>
+            <material name="red"/>
+        </visual>
+        <collision>
+            <geometry>
+                <box size="0.03 0.03 0.03"/>
+            </geometry>
+            <material name="red"/>
+        </collision>
+        <inertial>
+            <mass value="0.1"/>
+            <origin xyz="0 0 0" rpy="0 0 0"/>
+            <inertia ixx="0.0001" ixy="0.0" ixz="0.0" iyy="0.0001" iyz="0.0" izz="0.0001"/>
+        </inertial>
+    </link>
 </robot>
