Commit message: Included ros2_control

File: description/gazebo_control.xacro (robot description, xacro)
@@ -1,15 +1,15 @@
 <?xml version="1.0"?>
-<robot xmlns:xacro="http://www.ros.org/wiki/xacro" >
+<robot xmlns:xacro="http://www.ros.org/wiki/xacro">
     <gazebo>
         <plugin name="diff_drive" filename="libgazebo_ros_diff_drive.so">
-            <!--Wheel Information-->
+            <!-- Wheel Information -->
             <left_joint>left_wheel_joint</left_joint>
             <right_joint>right_wheel_joint</right_joint>
-            <wheel_seperation>0.35</wheel_seperation>
+            <wheel_separation>0.297</wheel_separation>
             <wheel_diameter>0.08</wheel_diameter>
-            <!--Limits-->
+            <!-- Limits -->
             <max_wheel_torque>200</max_wheel_torque>
-            <max_wheel_accleration>10.0</max_wheel_accleration>
-            <!--Output-->
+            <max_wheel_acceleration>10.0</max_wheel_acceleration>
+            <!-- Output -->
             <odometry_frame>odom</odometry_frame>
             <robot_base_frame>base_link</robot_base_frame>

File: description/robot.urdf.xacro (robot description, xacro)
@@ -2,5 +2,5 @@
 <robot xmlns:xacro="http://www.ros.org/wiki/xacro"  name="robot">
     <xacro:include filename="robot_core.xacro"/>
-    <xacro:include filename="gazebo_control.xacro"/>
+    <xacro:include filename="ros2_control.xacro"/>
     <xacro:include filename="lidar.xacro"/>
 </robot>

File: description/robot_core.xacro (robot description, xacro)
@@ -1,165 +1,150 @@
 <?xml version="1.0"?>
-<robot xmlns:xacro="http://www.ros.org/wiki/xacro"  name="robot">
+<robot xmlns:xacro="http://www.ros.org/wiki/xacro" >
     <xacro:include filename="inertial_macros.xacro"/>
-   <material name="white">
-        <color rgba="1 1 1 1"/>
-   </material>
+    <xacro:property name="chassis_length" value="0.15"/>
+    <xacro:property name="chassis_width" value="0.23"/>
+    <xacro:property name="chassis_height" value="0.06"/>
+    <xacro:property name="chassis_mass" value="1.0"/>
+    <xacro:property name="wheel_radius" value="0.04"/>
+    <xacro:property name="wheel_thickness" value="0.04"/>
+    <xacro:property name="wheel_mass" value="0.05"/>
+    <xacro:property name="wheel_offset_x" value="0.33"/>
+    <xacro:property name="wheel_offset_y" value="0.135"/>
+    <xacro:property name="wheel_offset_z" value="0.01"/>
+    <xacro:property name="caster_wheel_radius" value="0.01"/>
+    <xacro:property name="caster_wheel_mass" value="0.01"/>
+    <xacro:property name="caster_wheel_offset_x" value="0.075"/>
+    <xacro:property name="caster_wheel_offset_z" value="${wheel_offset_z - wheel_radius + caster_wheel_radius}"/>
+    <material name="white">
+        <color rgba="1 1 1 1" />
+    </material>
     <material name="orange">
         <color rgba="1 0.3 0.1 1"/>
-   </material>
-   <material name="blue">
-    <color rgba="0.2 0.2 1 1"/>
-   </material>
-   <material name="red">
-        <color rgba="1 0 0 1"/>
-   </material>
+    </material>
+    <material name="blue">
+        <color rgba="0.2 0.2 1 1"/>
+    </material>
     <material name="black">
         <color rgba="0 0 0 1"/>
-   </material>
-    <!---Base-LInk-->
-   <link name="base_link">
-   </link>
-   <!--Base FootPrint Link-->
-   <joint name="base_footprint_joint" type="fixed">
-    <parent link="base_link"/>
-    <child link="base_footprint"/>
-    <origin xyz="0 0 0" rpy="0 0 0"/>
-   </joint>
-   <link name="base_footprint">
-   </link>
-   <!---Chasis-LInk-->
-    <joint name="chasis_joint" type="fixed">
-    <parent link="base_link"/>
-    <child link="chasis"/>
-    <origin xyz="-0.13 0 0"/>
+    </material>
+    <material name="red">
+        <color rgba="1 0 0 1"/>
+    </material>
+    <!-- BASE LINK -->
+    <link name="base_link">
+    </link>
+    <!-- BASE_FOOTPRINT LINK -->
+    <joint name="base_footprint_joint" type="fixed">
+        <parent link="base_link"/>
+        <child link="base_footprint"/>
+        <origin xyz="0 0 0" rpy="0 0 0"/>
     </joint>
-    <link name="chasis">
+    <link name="base_footprint">
+    </link>
+    <!-- CHASSIS LINK -->
+    <joint name="chassis_joint" type="fixed">
+        <parent link="base_link"/>
+        <child link="chassis"/>
+        <origin xyz="${-wheel_offset_x} 0 ${-wheel_offset_z}"/>
+    </joint>
+    <link name="chassis">
         <visual>
-        <origin xyz="0.075 0 0.0315"/>
+            <origin xyz="${chassis_length/2} 0 ${chassis_height/2}"/>
             <geometry>
-                <box size="0.15 0.23 0.063"/>
+                <box size="${chassis_length} ${chassis_width} ${chassis_height}"/>
+            </geometry>
+            <material name="orange"/>
+        </visual>
+        <collision>
+            <origin xyz="${chassis_length/2} 0 ${chassis_height/2}"/>
+            <geometry>
+                <box size="${chassis_length} ${chassis_width} ${chassis_height}"/>
+            </geometry>
+        </collision>
+        <xacro:inertial_box mass="0.5" x="${chassis_length}" y="${chassis_width}" z="${chassis_height}">
+            <origin xyz="${chassis_length/2} 0 ${chassis_height/2}" rpy="0 0 0"/>
+        </xacro:inertial_box>
+    </link>
+    <gazebo reference="chassis">
+        <material>Gazebo/Orange</material>
+    </gazebo>
+    <!-- LEFT WHEEL LINK -->
+    <joint name="left_wheel_joint" type="continuous">
+        <parent link="base_link"/>
+        <child link="left_wheel"/>
+        <origin xyz="0 ${wheel_offset_y} 0" rpy="-${pi/2} 0 0" />
+        <axis xyz="0 0 1"/>
+    </joint>
+    <link name="left_wheel">
+        <visual>
+            <geometry>
+                <cylinder radius="${wheel_radius}" length="${wheel_thickness}"/>
+            </geometry>
+            <material name="blue"/>
+        </visual>
+        <collision>
+            <geometry>
+                <sphere radius="${wheel_radius}"/>
+            </geometry>
+        </collision>
+        <xacro:inertial_cylinder mass="${wheel_mass}" length="${wheel_thickness}" radius="${wheel_radius}">
+            <origin xyz="0 0 0" rpy="0 0 0"/>
+        </xacro:inertial_cylinder>
+    </link>
+    <gazebo reference="left_wheel">
+        <material>Gazebo/Blue</material>
+    </gazebo>
+    <!-- RIGHT WHEEL LINK -->
+    <joint name="right_wheel_joint" type="continuous">
+        <parent link="base_link"/>
+        <child link="right_wheel"/>
+        <origin xyz="0 ${-wheel_offset_y} 0" rpy="${pi/2} 0 0" />
+        <axis xyz="0 0 -1"/>
+    </joint>
+    <link name="right_wheel">
+        <visual>
+            <geometry>
+                <cylinder radius="${wheel_radius}" length="${wheel_thickness}"/>
+            </geometry>
+            <material name="blue"/>
+        </visual>
+        <collision>
+            <geometry>
+                <sphere radius="${wheel_radius}"/>
+            </geometry>
+        </collision>
+        <xacro:inertial_cylinder mass="${wheel_mass}" length="${wheel_thickness}" radius="${wheel_radius}">
+            <origin xyz="0 0 0" rpy="0 0 0"/>
+        </xacro:inertial_cylinder>
+    </link>
+    <gazebo reference="right_wheel">
+        <material>Gazebo/Blue</material>
+    </gazebo>
+    <!-- CASTER WHEEL LINK -->
+    <joint name="caster_wheel_joint" type="fixed">
+        <parent link="chassis"/>
+        <child link="caster_wheel"/>
+        <origin xyz="${caster_wheel_offset_x} 0 ${caster_wheel_offset_z}"/>
+    </joint>
+    <link name="caster_wheel">
+        <visual>
+            <geometry>
+                <sphere radius="${caster_wheel_radius}"/>
             </geometry>
             <material name="white"/>
         </visual>
         <collision>
-        <origin xyz="0.075 0 0.0315"/>
             <geometry>
-                <box size="0.15 0.23 0.063"/>
+                <sphere radius="${caster_wheel_radius}"/>
             </geometry>
-            <material name="white"/>
         </collision>
-        <xacro:inertial_box mass="0.5" x="0.15" y="0.23" z="0.063">
-            <origin xyz="0.075 0 0.0315" rpy="0 0 0"/>
-        </xacro:inertial_box>
-    </link>
-    <gazebo reference="chasis">
-        <material>Gazebo/White</material>
-    </gazebo>
-    <!--Left-Wheel-Link-->
-    <joint name="left_wheel_joint" type="continuous">
-        <parent link ="base_link"/>
-        <child link = "left_wheel"/>
-        <origin xyz="0 0.165 0" rpy="${pi/2} 0 0"/>
-        <axis xyz="0 0 1"/>
-    </joint>
-    <link name = "left_wheel">
-    <visual>
-        <geometry>
-            <cylinder radius="0.04" length="0.04"/>
-        </geometry>
-        <material name="blue"/>
-    </visual>
-    <collision>
-        <geometry>
-            <cylinder radius="0.04" length="0.04"/>
-        </geometry>
-        <material name="blue"/>
-    </collision>
-    <xacro:inertial_cylinder mass="0.1" length="0.04" radius="0.04">
-        <origin xyz="0 0 0" rpy="0 0 0"/>
-    </xacro:inertial_cylinder>
-    </link>
-    <gazebo reference="left_wheel">
-        <material>Gazebo/Blue</material>
-    </gazebo>
-    <!--Right-Wheel-Link-->
-    <joint name="right_wheel_joint" type="continuous">
-        <parent link ="base_link"/>
-        <child link = "right_wheel"/>
-        <origin xyz="0 -0.165 0" rpy="${pi/2} 0 0"/>
-        <axis xyz="0 0 1"/>
-    </joint>
-    <link name = "right_wheel">
-    <visual>
-        <geometry>
-            <cylinder radius="0.04" length="0.04"/>
-        </geometry>
-        <material name="blue"/>
-    </visual>
-    <collision>
-        <geometry>
-            <cylinder radius="0.04" length="0.04"/>
-        </geometry>
-        <material name="blue"/>
-    </collision>
-    <xacro:inertial_cylinder mass="0.1" length="0.04" radius="0.04">
-        <origin xyz="0 0 0" rpy="0 0 0"/>
-    </xacro:inertial_cylinder>
-    </link>
-    <gazebo reference="right_wheel">
-        <material>Gazebo/Blue</material>
-    </gazebo>
-    <!--Caster Wheel-->
-    <joint name="caster_wheel_joint" type="fixed">
-        <parent link="base_link"/>
-        <child link="caster_wheel"/>
-        <origin xyz="-0.13 0 -0.018"/>
-    </joint>
-    <link name="caster_wheel">
-    <visual>
-        <geometry>
-            <sphere radius="0.02"/>
-        </geometry>
-        <material name="black"/>
-    </visual>
-     <collision>
-        <geometry>
-            <sphere radius="0.02"/>
-        </geometry>
-        <material name="black"/>
-    </collision>
-    <xacro:inertial_sphere mass="0.1" radius="0.05">
-        <origin xyz="0 0 0" rpy="0 0 0"/>
-    </xacro:inertial_sphere>
+        <xacro:inertial_sphere mass="${caster_wheel_mass}" radius="${caster_wheel_radius}">
+            <origin xyz="0 0 0" rpy="0 0 0"/>
+        </xacro:inertial_sphere>
     </link>
     <gazebo reference="caster_wheel">
-        <material>Gazebo/Black</material>
+        <material>Gazebo/White</material>
         <mu1 value="0.001"/>
         <mu2 value="0.001"/>
     </gazebo>
-    <!-- IMU Sensor -->
-    <joint name="base_to_imu" type="fixed">
-        <parent link="base_link"/>
-        <child link="imu"/>
-        <origin xyz="0 0 0.1" rpy="0 0 0"/>
-    </joint>
-    <link name="imu">
-        <visual>
-            <geometry>
-                <box size="0.03 0.03 0.03"/>
-            </geometry>
-            <material name="red"/>
-        </visual>
-        <collision>
-            <geometry>
-                <box size="0.03 0.03 0.03"/>
-            </geometry>
-            <material name="red"/>
-        </collision>
-        <inertial>
-            <mass value="0.1"/>
-            <origin xyz="0 0 0" rpy="0 0 0"/>
-            <inertia ixx="0.0001" ixy="0.0" ixz="0.0" iyy="0.0001" iyz="0.0" izz="0.0001"/>
-        </inertial>
-    </link>
 </robot>
