Commit message: Some Changes

File: description/lidar.xacro (robot description, xacro)
@@ -2,5 +2,5 @@
 <robot xmlns:xacro="http://www.ros.org/wiki/xacro" >
     <joint name="laser_joint" type="fixed">
-        <parent link="chasis"/>
+        <parent link="base_link"/>
         <child link="laser_frame"/>
         <origin xyz="0.1 0 0.083" rpy="0 0 0"/>

Commit message: Updated urdf for original model

File: description/lidar.xacro (robot description, xacro)
@@ -4,5 +4,5 @@
         <parent link="base_link"/>
         <child link="laser_frame"/>
-        <origin xyz="0.1 0 0.083" rpy="0 0 0"/>
+        <origin xyz="-0.08 0 0.105" rpy="0 0 0"/>
     </joint>
     <link name="laser_frame">
@@ -18,5 +18,5 @@
             </geometry>
         </collision>
-        <xacro:inertial_cylinder mass="0.1" length="0.04" radius="0.05">
+        <xacro:inertial_cylinder mass="0.1" length="0.04" radius="0.035">
             <origin xyz="0 0 0" rpy="0 0 0"/>
         </xacro:inertial_cylinder>

File: description/robot_core.xacro (robot description, xacro)
@@ -2,17 +2,17 @@
 <robot xmlns:xacro="http://www.ros.org/wiki/xacro" >
     <xacro:include filename="inertial_macros.xacro"/>
-    <xacro:property name="chassis_length" value="0.15"/>
-    <xacro:property name="chassis_width" value="0.23"/>
-    <xacro:property name="chassis_height" value="0.06"/>
+    <xacro:property name="chassis_length" value="0.28"/>
+    <xacro:property name="chassis_width" value="0.2"/>
+    <xacro:property name="chassis_height" value="0.05"/>
     <xacro:property name="chassis_mass" value="1.0"/>
     <xacro:property name="wheel_radius" value="0.04"/>
     <xacro:property name="wheel_thickness" value="0.04"/>
     <xacro:property name="wheel_mass" value="0.05"/>
-    <xacro:property name="wheel_offset_x" value="0.33"/>
+    <xacro:property name="wheel_offset_x" value="0.265"/>
     <xacro:property name="wheel_offset_y" value="0.135"/>
-    <xacro:property name="wheel_offset_z" value="0.01"/>
-    <xacro:property name="caster_wheel_radius" value="0.01"/>
+    <xacro:property name="wheel_offset_z" value="-0.03"/>
+    <xacro:property name="caster_wheel_radius" value="0.025"/>
     <xacro:property name="caster_wheel_mass" value="0.01"/>
-    <xacro:property name="caster_wheel_offset_x" value="0.075"/>
+    <xacro:property name="caster_wheel_offset_x" value="0.05"/>
     <xacro:property name="caster_wheel_offset_z" value="${wheel_offset_z - wheel_radius + caster_wheel_radius}"/>
     <material name="white">

Commit message: Update

File: description/lidar.xacro (robot description, xacro)
@@ -4,5 +4,5 @@
         <parent link="base_link"/>
         <child link="laser_frame"/>
-        <origin xyz="0.1 0 0.083" rpy="0 0 0"/>
+        <origin xyz="-0.14 0 0.083" rpy="0 0 3.14159"/>
     </joint>
     <link name="laser_frame">

File: description/robot_core.xacro (robot description, xacro)
@@ -2,17 +2,17 @@
 <robot xmlns:xacro="http://www.ros.org/wiki/xacro" >
     <xacro:include filename="inertial_macros.xacro"/>
-    <xacro:property name="chassis_length" value="0.15"/>
-    <xacro:property name="chassis_width" value="0.23"/>
-    <xacro:property name="chassis_height" value="0.06"/>
+    <xacro:property name="chassis_length" value="0.28"/>
+    <xacro:property name="chassis_width" value="0.2"/>
+    <xacro:property name="chassis_height" value="0.05"/>
     <xacro:property name="chassis_mass" value="1.0"/>
     <xacro:property name="wheel_radius" value="0.04"/>
     <xacro:property name="wheel_thickness" value="0.04"/>
     <xacro:property name="wheel_mass" value="0.05"/>
-    <xacro:property name="wheel_offset_x" value="0.33"/>
+    <xacro:property name="wheel_offset_x" value="0.265"/>
     <xacro:property name="wheel_offset_y" value="0.135"/>
-    <xacro:property name="wheel_offset_z" value="0.01"/>
-    <xacro:property name="caster_wheel_radius" value="0.01"/>
+    <xacro:property name="wheel_offset_z" value="-0.03"/>
+    <xacro:property name="caster_wheel_radius" value="0.025"/>
     <xacro:property name="caster_wheel_mass" value="0.01"/>
-    <xacro:property name="caster_wheel_offset_x" value="0.075"/>
+    <xacro:property name="caster_wheel_offset_x" value="0.05"/>
     <xacro:property name="caster_wheel_offset_z" value="${wheel_offset_z - wheel_radius + caster_wheel_radius}"/>
     <material name="white">
@@ -73,5 +73,5 @@
         <parent link="base_link"/>
         <child link="left_wheel"/>
-        <origin xyz="0 ${wheel_offset_y} 0" rpy="-${pi/2} 0 0" />
+        <origin xyz="0 ${wheel_offset_y} 0" rpy="${pi/2} 0 0" />
         <axis xyz="0 0 1"/>
     </joint>
