Commit message: Added Lidar Xarco

File: description/robot.urdf.xacro (robot description, xacro)
@@ -3,3 +3,4 @@
     <xacro:include filename="robot_core.xacro"/>
     <xacro:include filename="gazebo_control.xacro"/>
+    <xacro:include filename="lidar.xacro"/>
 </robot>

File: description/robot_core.xacro (robot description, xacro)
@@ -11,5 +11,8 @@
     <color rgba="0.2 0.2 1 1"/>
    </material>
-   <material name="black">
+   <material name="red">
+        <color rgba="1 0 0 1"/>
+   </material>
+    <material name="black">
         <color rgba="0 0 0 1"/>
    </material>

Commit message: Final Sync

File: description/robot.urdf.xacro (robot description, xacro)
@@ -3,5 +3,4 @@
     <xacro:include filename="robot_core.xacro"/>
     <xacro:include filename="ros2_control.xacro"/>
-    <xacro:include filename="imu_sensor.xacro"/>
     <xacro:include filename="lidar.xacro"/>
 </robot>

File: description/robot_core.xacro (robot description, xacro)
@@ -73,5 +73,5 @@
         <parent link="base_link"/>
         <child link="left_wheel"/>
-        <origin xyz="0 ${wheel_offset_y} 0" rpy="${pi/2} 0 0" />
+        <origin xyz="0 ${wheel_offset_y} 0" rpy="-${pi/2} 0 0" />
         <axis xyz="0 0 1"/>
     </joint>

File: description/ros2_control.xacro (robot description, xacro)
@@ -8,5 +8,5 @@
                 <param name="loop_rate">30</param>
                 <param name="device">/dev/ttyACM0</param>
-                <param name="baud_rate">9600</param>
+                <param name="baud_rate">57600</param>
                 <param name="timeout">1000</param>
                 <param name="enc_counts_per_rev">1080</param>
